Commit message: update README and fix files

File: urdf/macros/link_igv.urdf.xacro (robot description, xacro)
@@ -3,59 +3,48 @@
   <!-- box -->
   <xacro:macro name="create_box" params="m x y z *origin">
-    <inertial>
-      <mass value="${m}" />
-      <inertia
-        ixx="${1/12*m*(y*y+z*z)}" ixy="0.0" ixz="0.0"
-        iyy="${1/12*m*(x*x+z*z)}" iyz="0.0"
-        izz="${1/12*m*(x*x+y*y)}" />
-    </inertial>
-    <collision>
-      <geometry>
-        <box size="${x} ${y} ${z}"/>
-      </geometry>
-    </collision>
     <visual>
+      <xacro:insert_block name="origin"/>
       <geometry>
         <box size="${x} ${y} ${z}"/>
       </geometry>
     </visual>
+    <!-- <collision>
+      <xacro:insert_block name="origin"/>
+      <geometry>
+        <box size="${x} ${y} ${z}"/>
+      </geometry>
+    </collision> -->
+    <!-- <inertial>
+      <mass value="${m}"/>
+      <inertia
+        ixx="${1/12*m*(y*y+z*z)}" ixy="0.0" ixz="0.0"
+        iyy="${1/12*m*(x*x+z*z)}" iyz="0.0"
+        izz="${1/12*m*(x*x+y*y)}"/>
+    </inertial> -->
   </xacro:macro>
   <!-- cylinder -->
   <xacro:macro name="create_cylinder" params="m r l *origin">
-    <inertial>
-      <mass value="${m}"/>
-      <inertia
-        ixx="${m*r*r}" ixy="0.0" ixz="0.0"
-        iyy="${m*r*r}" iyz="0.0"
-        izz="${m*r*r}"/>
-    </inertial>
-    <collision>
-      <xacro:insert_block name="origin" />
-      <geometry>
-        <cylinder radius="${r}" length="${l}"/>
-      </geometry>
-    </collision>
     <visual>
-      <xacro:insert_block name="origin" />
+      <xacro:insert_block name="origin"/>
       <geometry>
         <cylinder radius="${r}" length="${l}"/>
       </geometry>
     </visual>
+    <!-- <collision>
+      <xacro:insert_block name="origin"/>
+      <geometry>
+        <cylinder radius="${r}" length="${l}"/>
+      </geometry>
+    </collision> -->
+    <!-- <inertial>
+      <mass value="${m}"/>
+      <inertia
+        ixx="${1/12*m*(3*r*r+l*l)}" ixy="0.0" ixz="0.0"
+        iyy="${1/12*m*(3*r*r+l*l)}" iyz="0.0"
+        izz="${1/2*(m*r*r)}"/>
+    </inertial> -->
   </xacro:macro>
   <!-- sphere -->
   <xacro:macro name="create_sphere" params="m r *origin">
-    <inertial>
-      <mass value="${m}"/>
-      <inertia
-        ixx="${(2/5)*m*r*r}" ixy="0.0" ixz="0.0"
-        iyy="${(2/5)*m*r*r}" iyz="0.0"
-        izz="${(2/5)*m*r*r}"/>
-    </inertial>
-    <collision>
-      <xacro:insert_block name="origin" />
-      <geometry>
-        <sphere radius="${r}"/>
-      </geometry>
-    </collision>
     <visual>
       <xacro:insert_block name="origin" />
@@ -64,4 +53,17 @@
       </geometry>
     </visual>
+    <!-- <collision>
+      <xacro:insert_block name="origin" />
+      <geometry>
+        <sphere radius="${r}"/>
+      </geometry>
+    </collision> -->
+    <!-- <inertial>
+      <mass value="${m}"/>
+      <inertia
+        ixx="${(2/5)*m*r*r}" ixy="0.0" ixz="0.0"
+        iyy="${(2/5)*m*r*r}" iyz="0.0"
+        izz="${(2/5)*m*r*r}"/>
+    </inertial> -->
   </xacro:macro>
 </robot>

File: urdf/macros/parts/wheel.urdf.xacro (robot description, xacro)
@@ -4,5 +4,5 @@
     <!-- link: wheel -->
     <link name="${name}_wheel">
-      <origin rpy="${PI/2} 0 0"/>
+      <origin xyz="0 0 0" rpy="${PI/2} 0 0"/>
       <xacro:create_sphere m="1" r="${body_scale/20}">
         <origin xyz="0 0 0" rpy="0 0 0"/>

File: urdf/myfirstrobot.urdf.xacro (robot description, xacro)
@@ -7,6 +7,6 @@
   <xacro:include filename="$(find myfirstrobot_description)/urdf/macros/parts/head.urdf.xacro" />
   <xacro:include filename="$(find myfirstrobot_description)/urdf/macros/parts/leg.urdf.xacro" />
-  <xacro:include filename="$(find myfirstrobot_description)/urdf/simulation/gazebo_base.urdf.xacro" />
-  <xacro:include filename="$(find myfirstrobot_description)/urdf/simulation/gazebo_camera.urdf.xacro" />
+  <!-- <xacro:include filename="$(find myfirstrobot_description)/urdf/simulation/gazebo_base.urdf.xacro" /> -->
+  <!-- <xacro:include filename="$(find myfirstrobot_description)/urdf/simulation/gazebo_camera.urdf.xacro" /> -->
   <!-- Robot -->
   <xacro:base name="base"/>
@@ -19,5 +19,5 @@
   </xacro:leg>
   <!-- Plugins -->
-  <xacro:gazebo_base reference="base"/>
-  <xacro:gazebo_camera reference="head_box"/>
+  <!-- <xacro:gazebo_base reference="base"/> -->
+  <!-- <xacro:gazebo_camera reference="head_box"/> -->
 </robot>

File: urdf/simulation/gazebo_camera.urdf.xacro (robot description, xacro)
@@ -3,7 +3,6 @@
   <xacro:macro name="gazebo_camera" params="reference">
     <gazebo reference="${reference}">
-      <sensor type="camera" name="sensor_${reference}">
-        <update_rate>30.0</update_rate>
-        <camera name="camera_${reference}">
+      <sensor name="sensor_${reference}" type="camera">
+        <camera>
           <horizontal_fov>1.3962634</horizontal_fov>
           <image>
@@ -16,9 +15,4 @@
             <far>300</far>
           </clip>
-          <noise>
-            <type>gaussian</type>
-            <mean>0.0</mean>
-            <stddev>0.007</stddev>
-          </noise>
         </camera>
         <plugin name="${reference}_controller" filename="libgazebo_ros_camera.so">
