Commit message: parse to ros2

File: urdf/macros/link_geometry.urdf.xacro (robot description, xacro)
@@ -1,4 +1,7 @@
 <?xml version="1.0"?>
 <robot xmlns:xacro="http://ros.org/wiki/xacro">
+      <material name="Cyan">
+        <color rgba="0 1.0 1.0 1.0"/>
+      </material>
   <!-- box -->
   <xacro:macro name="create_box" params="m x y z *origin">
@@ -8,12 +11,13 @@
         <box size="${x} ${y} ${z}"/>
       </geometry>
+      <material name="Cyan"/>
     </visual>
-    <!-- <collision>
+    <collision>
       <xacro:insert_block name="origin"/>
       <geometry>
         <box size="${x} ${y} ${z}"/>
       </geometry>
-    </collision> -->
-    <!-- <inertial>
+    </collision>
+    <inertial>
       <mass value="${m}"/>
       <inertia
@@ -21,5 +25,5 @@
         iyy="${1/12*m*(x*x+z*z)}" iyz="0.0"
         izz="${1/12*m*(x*x+y*y)}"/>
-    </inertial> -->
+    </inertial>
   </xacro:macro>
   <!-- cylinder -->
@@ -30,12 +34,13 @@
         <cylinder radius="${r}" length="${l}"/>
       </geometry>
+      <material name="Cyan"/>
     </visual>
-    <!-- <collision>
+    <collision>
       <xacro:insert_block name="origin"/>
       <geometry>
         <cylinder radius="${r}" length="${l}"/>
       </geometry>
-    </collision> -->
-    <!-- <inertial>
+    </collision>
+    <inertial>
       <mass value="${m}"/>
       <inertia
@@ -43,5 +48,5 @@
         iyy="${1/12*m*(3*r*r+l*l)}" iyz="0.0"
         izz="${1/2*(m*r*r)}"/>
-    </inertial> -->
+    </inertial>
   </xacro:macro>
   <!-- sphere -->
@@ -53,11 +58,11 @@
       </geometry>
     </visual>
-    <!-- <collision>
+    <collision>
       <xacro:insert_block name="origin" />
       <geometry>
         <sphere radius="${r}"/>
       </geometry>
-    </collision> -->
-    <!-- <inertial>
+    </collision>
+    <inertial>
       <mass value="${m}"/>
       <inertia
@@ -65,5 +70,5 @@
         iyy="${(2/5)*m*r*r}" iyz="0.0"
         izz="${(2/5)*m*r*r}"/>
-    </inertial> -->
+    </inertial>
   </xacro:macro>
 </robot>

File: urdf/macros/parts/base.urdf.xacro (robot description, xacro)
@@ -4,4 +4,10 @@
     <!-- link: base_footprint -->
     <link name='base_footprint'/>
+    <!-- joint: base_footprint -> base -->
+    <joint name="joint_base_footprint_to_base" type="fixed">
+      <origin xyz="0 0 ${2*robot_scale/3}" rpy="0 0 0"/>
+      <parent link="base_footprint"/>
+      <child link="${name}"/>
+    </joint>
     <!-- link: base -->
     <link name="${name}">
@@ -10,10 +16,11 @@
       </xacro:create_cylinder>
     </link>
-    <!-- joint: base_footprint -> base -->
-    <joint name="joint_base_footprint_to_base" type="fixed">
-      <origin xyz="0 0 ${2*robot_scale/3}" rpy="0 0 0"/>
-      <parent link="base_footprint"/>
-      <child link="base"/>
-    </joint>
+  <joint name="base_to_laser" type="fixed">
+    <origin xyz="0 0 -0.3" rpy="0 0 0"/>
+    <parent link="${name}"/>
+    <child link="base_scan"/>
+  </joint>
+  <link name="base_scan">
+  </link>
   </xacro:macro>
 </robot>

File: urdf/macros/parts/leg.urdf.xacro (robot description, xacro)
@@ -3,4 +3,10 @@
   <xacro:include filename="$(find myfirstrobot_description)/urdf/macros/parts/wheel.urdf.xacro" />
   <xacro:macro name="leg" params="name parent *origin">
+    <!-- joint: parent -> leg -->
+    <joint name="${parent}_to_${name}_leg" type="fixed">
+      <xacro:insert_block name="origin" />
+      <parent link="${parent}"/>
+      <child link="${name}_leg"/>
+    </joint>
     <!-- link: leg -->
     <link name="${name}_leg">
@@ -9,4 +15,10 @@
       </xacro:create_box>
     </link>
+    <!-- joint: leg -> leg_base -->
+    <joint name="${name}_leg_to_${name}_leg_base" type="fixed">
+      <origin xyz="0 0 -${robot_scale/2}" rpy="0 0 0"/>
+      <parent link="${name}_leg"/>
+      <child link="${name}_leg_base"/>
+    </joint>
     <!-- link: leg_base -->
     <link name="${name}_leg_base">
@@ -15,23 +27,15 @@
       </xacro:create_box>
     </link>
-    <!-- joint: parent -> leg -->
-    <joint name="${parent}_to_${name}_leg" type="fixed">
-      <xacro:insert_block name="origin" />
-      <parent link="${parent}"/>
-      <child link="${name}_leg"/>
-    </joint>
-    <!-- joint: leg -> leg_base -->
-    <joint name="${name}_leg_to_${name}_leg_base" type="fixed">
-      <origin xyz="0 0 -${robot_scale/2}" rpy="0 0 0"/>
-      <parent link="${name}_leg"/>
-      <child link="${name}_leg_base"/>
-    </joint>
     <!-- front wheel -->
     <xacro:wheel name="${name}_front_wheel" parent="${name}_leg_base">
-      <origin xyz="${robot_scale/5} 0 -${robot_scale/10}" rpy="0 0 0"/>
+      <origin xyz="${robot_scale/5} 0 -${robot_scale/10}" rpy="-1.57 0 0"/>
+    </xacro:wheel>
+    <!-- center wheel -->
+    <xacro:wheel name="${name}_center_wheel" parent="${name}_leg_base">
+      <origin xyz="0 0 -${robot_scale/10 + 0.001}" rpy="-1.57 0 0"/>
     </xacro:wheel>
     <!-- back wheel -->
     <xacro:wheel name="${name}_back_wheel" parent="${name}_leg_base">
-      <origin xyz="-${robot_scale/5} 0 -${robot_scale/10}" rpy="0 0 0"/>
+      <origin xyz="-${robot_scale/5} 0 -${robot_scale/10}" rpy="-1.57 0 0"/>
     </xacro:wheel>
   </xacro:macro>

File: urdf/macros/parts/wheel.urdf.xacro (robot description, xacro)
@@ -2,18 +2,18 @@
 <robot xmlns:xacro="http://ros.org/wiki/xacro">
   <xacro:macro name="wheel" params="name parent *origin">
+    <!-- joint: parent_base -> wheel -->
+    <joint name="${parent}_to_${name}" type="continuous">
+      <xacro:insert_block name="origin" />
+      <parent link="${parent}"/>
+      <child link="${name}"/>
+      <axis xyz="0 0 1"/>
+    </joint>
     <!-- link: wheel -->
-    <link name="${name}_wheel">
-      <origin xyz="0 0 0" rpy="${PI/2} 0 0"/>
+    <link name="${name}">
+      <origin xyz="0 0 0" rpy="${-PI/2} 0 0"/>
       <xacro:create_sphere m="${wheel_mass}" r="${wheel_radius}">
         <origin xyz="0 0 0" rpy="0 0 0"/>
       </xacro:create_sphere>
     </link>
-    <!-- joint: parent_base -> wheel -->
-    <joint name="${parent}_to_${name}_wheel" type="continuous">
-      <xacro:insert_block name="origin" />
-      <parent link="${parent}"/>
-      <child link="${name}_wheel"/>
-      <axis xyz="0 1 0"/>
-    </joint>
   </xacro:macro>
 </robot>

File: urdf/myfirstrobot.urdf (robot description, URDF)
Before this commit: robot myfirstrobot, 12 links, 11 joints
Links:
- link base_footprint: geometry 

File: urdf/myfirstrobot.urdf.xacro (robot description, xacro)
@@ -7,17 +7,19 @@
   <xacro:include filename="$(find myfirstrobot_description)/urdf/macros/parts/head.urdf.xacro" />
   <xacro:include filename="$(find myfirstrobot_description)/urdf/macros/parts/leg.urdf.xacro" />
-  <!-- <xacro:include filename="$(find myfirstrobot_description)/urdf/simulation/gazebo_base.urdf.xacro" /> -->
-  <!-- <xacro:include filename="$(find myfirstrobot_description)/urdf/simulation/gazebo_camera.urdf.xacro" /> -->
+  <xacro:include filename="$(find myfirstrobot_description)/urdf/simulation/gazebo_base.urdf.xacro" />
+  <xacro:include filename="$(find myfirstrobot_description)/urdf/simulation/gazebo_laser.urdf.xacro" />
+  <xacro:include filename="$(find myfirstrobot_description)/urdf/simulation/gazebo_camera.urdf.xacro" />
   <!-- Robot -->
-  <xacro:base name="base"/>
-  <xacro:head name="head" parent="base"/>
-  <xacro:leg name="right" parent="base">
+  <xacro:base name="base_link"/>
+  <xacro:head name="head" parent="base_link"/>
+  <xacro:leg name="left" parent="base_link">
     <origin xyz="0  ${robot_scale/3} -${robot_scale/10}" rpy="0 0 0"/>
   </xacro:leg>
-  <xacro:leg name="left" parent="base">
+  <xacro:leg name="right" parent="base_link">
     <origin xyz="0 -${robot_scale/3} -${robot_scale/10}" rpy="0 0 0"/>
   </xacro:leg>
   <!-- Plugins -->
-  <!-- <xacro:gazebo_base reference="base"/> -->
-  <!-- <xacro:gazebo_camera reference="head_box"/> -->
+  <xacro:gazebo_base/>
+  <xacro:gazebo_laser reference="base_scan"/>
+  <xacro:gazebo_camera reference="head_box"/>
 </robot>

File: urdf/simulation/gazebo_base.urdf.xacro (robot description, xacro)
@@ -1,13 +1,40 @@
 <?xml version="1.0"?>
 <robot xmlns:xacro="http://ros.org/wiki/xacro">
-  <xacro:macro name="gazebo_base" params="reference">
+  <xacro:macro name="gazebo_base">
     <gazebo>
-      <plugin name="${reference}_controller" filename="libgazebo_ros_planar_move.so">
-        <commandTopic>cmd_vel</commandTopic>
-        <odometryTopic>odom</odometryTopic>
-        <odometryFrame>odom</odometryFrame>
-        <odometryRate>100.0</odometryRate>
-        <robotBaseFrame>${reference}_footprint</robotBaseFrame>
+      <plugin name='diff_drive' filename='libgazebo_ros_diff_drive.so'>
+        <ros>
+          <!-- <namespace>/r2d2</namespace> -->
+          <!-- <remapping>cmd_vel:=cmd_vel</remapping> -->
+          <!-- <remapping>odom:=odom</remapping> -->
+        </ros>
+        <update_rate>30</update_rate>
+        <command_topic>cmd_vel</command_topic>
+        <!-- wheels -->
+        <left_joint>left_leg_base_to_left_center_wheel</left_joint>
+        <right_joint>right_leg_base_to_right_center_wheel</right_joint>
+        <!-- kinematics -->
+        <wheel_separation>0.4</wheel_separation>
+        <wheel_diameter>0.04</wheel_diameter>
+        <!-- limits -->
+        <max_wheel_torque>20</max_wheel_torque>
+        <max_wheel_acceleration>1.0</max_wheel_acceleration>
+        <!-- output -->
+        <publish_odom>true</publish_odom>
+        <publish_odom_tf>true</publish_odom_tf>
+        <publish_wheel_tf>false</publish_wheel_tf>
+        <odometry_topic>odom</odometry_topic>
+        <odometry_frame>odom</odometry_frame>
+        <robot_base_frame>base_footprint</robot_base_frame>
       </plugin>
+    <!-- <plugin name="joint_state" filename="libgazebo_ros_joint_state_publisher.so">
+      <ros>
+        <remapping>~/out:=joint_states</remapping>
+      </ros>
+      <update_rate>30</update_rate>
+      <joint_name>left_leg_base_to_left_center_wheel</joint_name>
+      <joint_name>right_leg_base_to_right_center_wheel</joint_name>
+      <joint_name>joint_base_footprint_to_base</joint_name>
+    </plugin>   -->
     </gazebo>
   </xacro:macro>

File: urdf/simulation/gazebo_camera.urdf.xacro (robot description, xacro)
@@ -3,5 +3,5 @@
   <xacro:macro name="gazebo_camera" params="reference">
     <gazebo reference="${reference}">
-      <sensor name="sensor_${reference}" type="camera">
+      <!-- <sensor name="sensor_${reference}" type="camera">
         <camera>
           <horizontal_fov>1.3962634</horizontal_fov>
@@ -30,5 +30,36 @@
           <distortionT2>0.0</distortionT2>
         </plugin>
-      </sensor>
+      </sensor> -->
+            <sensor type="camera" name="camera1">
+          <update_rate>60</update_rate>
+          <visualize>true</visualize>
+          <camera name="head">
+            <horizontal_fov>1.3962634</horizontal_fov>
+            <image>
+              <width>640</width>
+              <height>480</height>
+              <format>R8G8B8</format>
+            </image>
+            <clip>
+              <near>0.02</near>
+              <far>300</far>
+            </clip>
+            <noise>
+              <type>gaussian</type>
+              <mean>0.0</mean>
+              <stddev>0.007</stddev>
+            </noise>
+          </camera>
+          <plugin name="camera_controller" filename="libgazebo_ros_camera.so">
+            <ros>
+              <namespace>r2d2</namespace>
+              <!-- TODO(louise) Remapping not working due to https://github.com/ros-perception/image_common/issues/93 -->
+              <!-- <remapping>image_raw:=image_demo</remapping> -->
+              <!-- <remapping>camera_info:=camera_info_demo</remapping> -->
+            </ros>
+            <!-- camera_name>omit so it defaults to sensor name</camera_name-->
+            <!-- frame_name>omit so it defaults to link name</frame_name-->
+          </plugin>
+        </sensor>
     </gazebo>
   </xacro:macro>
