Commit message: update README and properties

File: urdf/macros/parts/base.urdf.xacro (robot description, xacro)
@@ -6,5 +6,5 @@
     <!-- link: base -->
     <link name="${name}">
-      <xacro:create_cylinder m="2" r="${body_scale/3}" l="${body_scale}">
+      <xacro:create_cylinder m="${body_mass}" r="${body_radius}" l="${body_length}">
         <origin xyz="0 0 0" rpy="0 0 0"/>
       </xacro:create_cylinder>
@@ -12,5 +12,5 @@
     <!-- joint: base_footprint -> base -->
     <joint name="joint_base_footprint_to_base" type="fixed">
-      <origin xyz="0 0 ${2*body_scale/3}" rpy="0 0 0"/>
+      <origin xyz="0 0 ${2*robot_scale/3}" rpy="0 0 0"/>
       <parent link="base_footprint"/>
       <child link="base"/>

File: urdf/macros/parts/head.urdf.xacro (robot description, xacro)
@@ -1,8 +1,9 @@
 <?xml version="1.0"?>
 <robot xmlns:xacro="http://ros.org/wiki/xacro">
+  <xacro:property name="robot_scale" value="0.6" />
     <xacro:macro name="head" params="name parent">
       <!-- link: head -->
       <link name="${name}">
-        <xacro:create_sphere m="1" r="${body_scale/3}">
+        <xacro:create_sphere m="${head_mass}" r="${head_radius}">
           <origin xyz="0 0 0" rpy="0 0 0"/>
         </xacro:create_sphere>
@@ -10,5 +11,5 @@
       <!-- link: head_box -->
       <link name="${name}_box">
-        <xacro:create_box m="1" x="${body_scale/10}" y="${body_scale/10}" z="${body_scale/10}">
+        <xacro:create_box m="${head_mass/100}" x="${head_radius/3}" y="${head_radius/3}" z="${head_radius/3}">
           <origin xyz="0 0 0" rpy="0 0 0"/>
         </xacro:create_box>
@@ -16,13 +17,13 @@
       <!-- joint: base -> head -->
       <joint name="joint_${parent}_to_${name}" type="revolute">
-        <origin xyz="0 0 ${body_scale/2}" rpy="0 0 0"/>
+        <origin xyz="0 0 ${robot_scale/2}" rpy="0 0 0"/>
         <parent link="${parent}"/>
         <child link="${name}"/>
         <axis xyz="0 0 1"/>
-        <limit effort="${effort}" velocity="${velocity}" lower="-${PI/2}" upper="${PI/2}"/>
+        <limit effort="30" velocity="0.5" lower="-${PI/2}" upper="${PI/2}"/>
       </joint>
       <!-- joint: head -> head_box -->
-      <joint name="joint_head_to_head_box" type="fixed">
-        <origin xyz="${body_scale/5} 0 ${body_scale/4}" rpy="0 0 0"/>
+      <joint name="joint_${name}_to_${name}_box" type="fixed">
+        <origin xyz="${robot_scale/5} 0 ${robot_scale/4}" rpy="0 0 0"/>
         <parent link="${name}"/>
         <child link="${name}_box"/>

File: urdf/macros/parts/leg.urdf.xacro (robot description, xacro)
@@ -5,5 +5,5 @@
     <!-- link: leg -->
     <link name="${name}_leg">
-      <xacro:create_box m="1" x="${body_scale/3}" y="${body_scale/6}" z="${body_scale}">
+      <xacro:create_box m="${leg_mass}" x="${leg_x}" y="${leg_y}" z="${leg_z}">
         <origin xyz="0 0 0" rpy="0 0 0"/>
       </xacro:create_box>
@@ -11,5 +11,5 @@
     <!-- link: leg_base -->
     <link name="${name}_leg_base">
-      <xacro:create_box m="1" x="${2*body_scale/3}" y="${body_scale/6}" z="${body_scale/6}">
+      <xacro:create_box m="${leg_base_mass}" x="${2*robot_scale/3}" y="${robot_scale/6}" z="${robot_scale/6}">
         <origin xyz="0 0 0" rpy="0 0 0"/>
       </xacro:create_box>
@@ -23,5 +23,5 @@
     <!-- joint: leg -> leg_base -->
     <joint name="${name}_leg_to_${name}_leg_base" type="fixed">
-      <origin xyz="0 0 -${body_scale/2}" rpy="0 0 0"/>
+      <origin xyz="0 0 -${robot_scale/2}" rpy="0 0 0"/>
       <parent link="${name}_leg"/>
       <child link="${name}_leg_base"/>
@@ -29,9 +29,9 @@
     <!-- front wheel -->
     <xacro:wheel name="${name}_front_wheel" parent="${name}_leg_base">
-      <origin xyz="${body_scale/5} 0 -${body_scale/10}" rpy="0 0 0"/>
+      <origin xyz="${robot_scale/5} 0 -${robot_scale/10}" rpy="0 0 0"/>
     </xacro:wheel>
     <!-- back wheel -->
     <xacro:wheel name="${name}_back_wheel" parent="${name}_leg_base">
-      <origin xyz="-${body_scale/5} 0 -${body_scale/10}" rpy="0 0 0"/>
+      <origin xyz="-${robot_scale/5} 0 -${robot_scale/10}" rpy="0 0 0"/>
     </xacro:wheel>
   </xacro:macro>

File: urdf/macros/parts/wheel.urdf.xacro (robot description, xacro)
@@ -5,5 +5,5 @@
     <link name="${name}_wheel">
       <origin xyz="0 0 0" rpy="${PI/2} 0 0"/>
-      <xacro:create_sphere m="1" r="${body_scale/20}">
+      <xacro:create_sphere m="${wheel_mass}" r="${wheel_radius}">
         <origin xyz="0 0 0" rpy="0 0 0"/>
       </xacro:create_sphere>

File: urdf/macros/properties.urdf.xacro (robot description, xacro)
@@ -1,7 +1,21 @@
 <?xml version="1.0"?>
 <robot xmlns:xacro="http://ros.org/wiki/xacro">
-  <xacro:property name="PI"         value="3.14159265" />
-  <xacro:property name="body_scale" value="0.6" />
-  <xacro:property name="effort"     value="30" />
-  <xacro:property name="velocity"   value="0.5" />
+  <xacro:property name="PI"             value="3.14159265" />
+  <xacro:property name="robot_scale"     value="1.0" />
+  <xacro:property name="robot_mass"      value="10" />
+  <xacro:property name="body_mass"      value="${35 * robot_mass/100}" />
+  <xacro:property name="body_radius"    value="${robot_scale/3}" />
+  <xacro:property name="body_length"    value="${robot_scale}" />
+  <xacro:property name="head_mass"      value="${5 * robot_mass/100}" />
+  <xacro:property name="head_radius"    value="${body_radius}" />
+  <xacro:property name="leg_mass"       value="${5 * robot_mass/100}" />
+  <xacro:property name="leg_x"          value="${robot_scale/3}" />
+  <xacro:property name="leg_y"          value="${robot_scale/6}" />
+  <xacro:property name="leg_z"          value="${robot_scale}" />
+  <xacro:property name="leg_base_mass"  value="${15 * robot_mass/100}" />
+  <xacro:property name="leg_base_x"     value="${2*robot_scale/3}" />
+  <xacro:property name="leg_base_y"     value="${robot_scale/6}" />
+  <xacro:property name="leg_base_z"     value="${robot_scale/6}" />
+  <xacro:property name="wheel_mass"      value="${5 * robot_mass/100}" />
+  <xacro:property name="wheel_radius"    value="${body_radius/10}" />
 </robot>

File: urdf/myfirstrobot.urdf.xacro (robot description, xacro)
@@ -2,5 +2,5 @@
 <robot name="myfirstrobot"
   xmlns:xacro="http://www.ros.org/wiki/xacro">
-  <xacro:include filename="$(find myfirstrobot_description)/urdf/macros/link_igv.urdf.xacro" />
+  <xacro:include filename="$(find myfirstrobot_description)/urdf/macros/link_geometry.urdf.xacro" />
   <xacro:include filename="$(find myfirstrobot_description)/urdf/macros/properties.urdf.xacro" />
   <xacro:include filename="$(find myfirstrobot_description)/urdf/macros/parts/base.urdf.xacro" />
@@ -13,8 +13,8 @@
   <xacro:head name="head" parent="base"/>
   <xacro:leg name="right" parent="base">
-    <origin xyz="0  ${body_scale/3} -${body_scale/10}" rpy="0 0 0"/>
+    <origin xyz="0  ${robot_scale/3} -${robot_scale/10}" rpy="0 0 0"/>
   </xacro:leg>
   <xacro:leg name="left" parent="base">
-    <origin xyz="0 -${body_scale/3} -${body_scale/10}" rpy="0 0 0"/>
+    <origin xyz="0 -${robot_scale/3} -${robot_scale/10}" rpy="0 0 0"/>
   </xacro:leg>
   <!-- Plugins -->
